Commit message: making changes

File: prius_description/urdf/prius.urdf (robot description, URDF)
Before this commit: robot prius, 28 links, 27 joints
Links:
- added link dummy
Joints:
- added joint dummy_joint: type fixed, parent dummy, child base_link
- joint front_camera_joint: origin xyz=0 -0.4 1.4 rpy=0 0.05 -1.5707 -> xyz=0 -0.9 1.1 rpy=0 0 -1.5707
- joint front_left_laser_joint: origin xyz=1 -2.3 0.5 rpy=0 0.05 0 -> xyz=1 -1.9 0.5 rpy=0 0.05 0
- joint front_right_laser_joint: origin xyz=-1 -2.3 0.5 rpy=0 0.05 3.14 -> xyz=-1 -1.9 0.5 rpy=0 0.05 3.14

Commit message: updating urdf for IMU and GPS

File: prius_description/urdf/prius.urdf (robot description, URDF)
Before this commit: robot prius, 29 links, 28 joints
Links:
- added link gps_link, mass 1
- added link imu_link, mass 1
Joints:
- added joint gps_joint: type fixed, parent chassis, child gps_link, origin xyz=0.0 0.0 0.0 rpy=0 0 0
- added joint imu_joint: type fixed, parent chassis, child imu_link, origin xyz=0.0 0.0 0.0 rpy=0 0 0
